Commit message: fix bug

File: omniisaacgymenvs/assests/robots/ur16e/ur16e.urdf (robot description, URDF)
Before this commit: robot ur, 13 links, 12 joints
Links:
- removed link epick_end_effector
- removed link epick_rod
- removed link gripper_link
Joints:
- removed joint ee_fixed_joint
- removed joint eef_hand_joint
- removed joint gripper_joint
- joint rod_joint: child epick_rod -> ee_link; origin xyz=0 0 0.13 rpy=0 0 0 -> xyz=0 0 0.0 rpy=0 -1.57 0; parent gripper_link -> wrist_3_link

Commit message: Added Tacking objects

File: omniisaacgymenvs/assests/robots/ur16e/ur16e.urdf (robot description, URDF)
Before this commit: robot ur, 10 links, 9 joints
Links:
- added link sensor_1_link; visual cylinder length=0.01 radius=0.01
- added link sensor_2_link; visual cylinder length=0.01 radius=0.01
Joints:
- added joint sensor_1_joint: type fixed, parent wrist_3_link, child sensor_1_link, origin xyz=0.0323088 0 0.0768096 rpy=0 0 0
- added joint sensor_2_joint: type fixed, parent wrist_3_link, child sensor_2_link, origin xyz=-0.0323088 0 0.0768096 rpy=0 0 0
